File: Fluke_LCD/Fluke_LCD.kicad_sch (KiCad schematic)
At the start: 65 parts, among them J1 Conn_01x23

Commit message: A drop-in replacement now. Almost finished.
Parts:
- J1: footprint Connector_PinHeader_1.00mm:PinHeader_1x22_P1.00mm_Vertical -> FlukeLibrary:Fluke_8060A_LCD_ElastoPads
Changed lines of the file:
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@@
       (effects (font (size 1.27 1.27)))
     )
-    (property "Footprint" "Connector_PinHeader_1.00mm:PinHeader_1x22_P1.00mm_Vertical" (at 124.46 189.23 0)
+    (property "Footprint" "FlukeLibrary:Fluke_8060A_LCD_ElastoPads" (at 124.46 189.23 0)
       (effects (font (size 1.27 1.27)) hide)
     )

Commit message: Update libraries, positions, and footprints.
Parts:
- D1, D10, D11, D12, D13, D14, D15, D16, D17, D18, D19, D2, D20, D21, D22, D23, D24, D25, D26, D27, D28, D29, D3, D30, D31, D32, D33, D34, D35, D36, D38, D39, D4, D40, D41, D42, D43, D44, D5, D6, D7, D8, D9: footprint LED_SMD:LED_0805_2012Metric_Pad1.15x1.40mm_HandSolder -> FlukeLibrary:LED_0805_2012Metric_Pad1.3x1.40mm_HandSolder
