File: Fluke_LCD/Fluke_LCD.kicad_pcb (KiCad board)
At the start: 2 copper layers, 64.3 x 34 mm, 65 parts, among them J1 Conn_01x23

Commit message: A drop-in replacement now. Almost finished.
Parts:
- D1: value .1 -> 8A
- D10, D13: value 8A -> 8B
- D11, D14: value 8C -> 8B
- D17: value .1 -> 8C
- D18, D21: value 8A -> 8C
- D2, D3: value 8C -> 8A
- D20, D23: value 8B -> 8C
- D25: value .1 -> 8D
- D26, D29: value 8A -> 8D
- D27, D30: value 8C -> 8D
- D28, D31: value 8B -> 8D
- D4, D6: value 8B -> 8A
- D9: value .1 -> 8B
- J1: footprint Connector_PinHeader_1.00mm:PinHeader_1x22_P1.00mm_Vertical -> FlukeLibrary:Fluke_8060A_LCD_ElastoPads; moved to F.Cu
- moved J1 93.9 mm to (212.0, 145.0), turned to 0 degrees
- moved D42 88.9 mm to (189.0, 142.4)
- moved D40 87.0 mm to (192.3, 133.4), turned to 0 degrees
- moved D41 84.6 mm to (191.9, 139.4), turned to -90 degrees
- moved D38 84.5 mm to (202.6, 133.4)
- moved D43 84.4 mm to (191.9, 145.4), turned to -90 degrees
- moved D44 84.4 mm to (194.4, 149.5)
- moved D39 84.2 mm to (198.1, 133.4)
- moved D8 82.6 mm to (205.4, 149.5)
- moved D6 82.5 mm to (202.5, 145.4)
- moved D3 82.5 mm to (202.5, 139.3)
- moved D4 82.5 mm to (199.9, 142.4)
- moved D5 82.5 mm to (197.4, 145.4)
- moved D7 82.5 mm to (199.9, 148.5)
- moved D1 82.5 mm to (197.4, 139.3)
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Routing:
- net /TopGround: track 154.8 -> 227.0 mm, vias 0 -> 1
- net Net-(J1-Pin_4): track 45.3 -> 3.06 mm
- net Net-(J1-Pin_21): track 44.8 -> 3.02 mm
- net Net-(J1-Pin_19): track 43.3 -> 3.08 mm, vias 3 -> 1
- net Net-(J1-Pin_6): track 43.0 -> 3.03 mm
- net Net-(J1-Pin_5): track 42.9 -> 3.04 mm
- net Net-(J1-Pin_7): track 41.9 -> 3.04 mm
- net Net-(J1-Pin_2): track 41.9 -> 3.27 mm
- net Net-(J1-Pin_20): track 41.4 -> 3.06 mm
- net Net-(J1-Pin_22): track 41.2 -> 3.06 mm, vias 8 -> 1
- net Net-(J1-Pin_3): track 40.9 -> 3.08 mm
- net Net-(J1-Pin_8): track 40.0 -> 3.04 mm
- net Net-(J1-Pin_13): track 37.5 -> 3.04 mm, vias 4 -> 1
- net Net-(J1-Pin_9): track 36.8 -> 3.03 mm
- net Net-(J1-Pin_18): track 36.3 -> 3.04 mm, vias 3 -> 1
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
Commit message: Update libraries, positions, and footprints.
Parts:
- D1: value 8A -> .1; footprint LED_SMD:LED_0805_2012Metric_Pad1.15x1.40mm_HandSolder -> FlukeLibrary:LED_0805_2012Metric_Pad1.3x1.40mm_HandSolder
- D10, D13: value 8B -> 8A; footprint LED_SMD:LED_0805_2012Metric_Pad1.15x1.40mm_HandSolder -> FlukeLibrary:LED_0805_2012Metric_Pad1.3x1.40mm_HandSolder
- D11, D14: value 8B -> 8C; footprint LED_SMD:LED_0805_2012Metric_Pad1.15x1.40mm_HandSolder -> FlukeLibrary:LED_0805_2012Metric_Pad1.3x1.40mm_HandSolder
- D12, D15, D16, D19, D22, D24, D32, D33, D34, D35, D36, D38, D39, D40, D41, D42, D43, D44, D5, D7, D8: footprint LED_SMD:LED_0805_2012Metric_Pad1.15x1.40mm_HandSolder -> FlukeLibrary:LED_0805_2012Metric_Pad1.3x1.40mm_HandSolder
- D17: value 8C -> .1; footprint LED_SMD:LED_0805_2012Metric_Pad1.15x1.40mm_HandSolder -> FlukeLibrary:LED_0805_2012Metric_Pad1.3x1.40mm_HandSolder
- D18, D21: value 8C -> 8A; footprint LED_SMD:LED_0805_2012Metric_Pad1.15x1.40mm_HandSolder -> FlukeLibrary:LED_0805_2012Metric_Pad1.3x1.40mm_HandSolder
- D2, D3: value 8A -> 8C; footprint LED_SMD:LED_0805_2012Metric_Pad1.15x1.40mm_HandSolder -> FlukeLibrary:LED_0805_2012Metric_Pad1.3x1.40mm_HandSolder
- D20, D23: value 8C -> 8B; footprint LED_SMD:LED_0805_2012Metric_Pad1.15x1.40mm_HandSolder -> FlukeLibrary:LED_0805_2012Metric_Pad1.3x1.40mm_HandSolder
- D25: value 8D -> .1; footprint LED_SMD:LED_0805_2012Metric_Pad1.15x1.40mm_HandSolder -> FlukeLibrary:LED_0805_2012Metric_Pad1.3x1.40mm_HandSolder
- D26, D29: value 8D -> 8A; footprint LED_SMD:LED_0805_2012Metric_Pad1.15x1.40mm_HandSolder -> FlukeLibrary:LED_0805_2012Metric_Pad1.3x1.40mm_HandSolder
- D27, D30: value 8D -> 8C; footprint LED_SMD:LED_0805_2012Metric_Pad1.15x1.40mm_HandSolder -> FlukeLibrary:LED_0805_2012Metric_Pad1.3x1.40mm_HandSolder
- D28, D31: value 8D -> 8B; footprint LED_SMD:LED_0805_2012Metric_Pad1.15x1.40mm_HandSolder -> FlukeLibrary:LED_0805_2012Metric_Pad1.3x1.40mm_HandSolder
- D4, D6: value 8A -> 8B; footprint LED_SMD:LED_0805_2012Metric_Pad1.15x1.40mm_HandSolder -> FlukeLibrary:LED_0805_2012Metric_Pad1.3x1.40mm_HandSolder
- D9: value 8B -> .1; footprint LED_SMD:LED_0805_2012Metric_Pad1.15x1.40mm_HandSolder -> FlukeLibrary:LED_0805_2012Metric_Pad1.3x1.40mm_HandSolder
- moved J1 0.09 mm to (212.1, 145.0)
- moved D19 0.05 mm to (221.9, 136.2)
Routing:
- net /BottomGround: track 203.9 -> 200.3 mm

Commit message: 8060A LED Mod Rev1
Parts:
- added G***: LOGO, FlukeLibrary:johnflukenewerlogo_tiny_footprint, B.Cu at (192.2, 132.6)
Other:
- board text added: "8060A LED Mod Rev. 1 - Thanks to all at EEVBlog and ModemHead Inspired by Dmitri and the original LED 8060A Mod PCB Made by Parabolic Labs"
Changed lines of the file:
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@@
 			(drillshape 0)
 			(scaleselection 1)
-			(outputdirectory "output/")
+			(outputdirectory "pcb_output/")
 		)
 	)
@@
 		)
 	)
-	(gr_poly
-		(pts
-			(xy 239.117726 151.365) (xy 237.117726 131.365) (xy 187.117726 131.365) (xy 185.117726 151.365)
+	(footprint "FlukeLibrary:johnflukenewerlogo_tiny_footprint"
+		(layer "B.Cu")
+		(at 192.17 132.55 180)
+		(property "Reference" "G***"
+			(at -0.04 -5.35 360)
+			(layer "B.SilkS")
+			(hide yes)
+			(effects
+				(font
+					(size 1.5 1.5)
+					(thickness 0.3)
+				)
+				(justify mirror)
+			)
 		)
-		(stroke
-			(width 0.2)
-			(type dash_dot_dot)
+		(property "Value" "LOGO"
+			(at 0.02 4.86 360)
+			(layer "B.SilkS")
+			(hide yes)
+			(effects
+				(font
+					(size 1.5 1.5)
+					(thickness 0.3)
+				)
+				(justify mirror)
+			)
+		)
+		(property "Footprint" "FlukeLibrary:johnflukenewerlogo_tiny_footprint"
+			(at 0 0 360)
+			(layer "B.Fab")
+			(hide yes)
+			(effects
+				(font
+					(size 1.27 1.27)
+					(thickness 0.15)
+				)
+				(justify mirror)
+			)
+		)
+		(property "Datasheet" ""
+			(at 0 0 360)
+			(layer "B.Fab")
+			(hide yes)
+			(effects
+				(font
+					(size 1.27 1.27)
+					(thickness 0.15)
+				)
+				(justify mirror)
+			)
+		)
+		(property "Description" ""
+			(at 0 0 360)
+			(layer "B.Fab")
+			(hide yes)
+			(effects
+				(font
+					(size 1.27 1.27)
+					(thickness 0.15)
+				)
+				(justify mirror)
+			)
+		)
+		(attr board_only exclude_from_pos_files exclude_from_bom)
+		(fp_rect
+			(start 2.278305 2.555672)
+			(end 2.92 -0.235672)
+			(stroke
+				(width 0)
+				(type solid)
+			)
+			(fill solid)
+			(layer "B.SilkS")
+		)
+		(fp_rect
+			(start 0.808305 2.551344)
+			(end 1.45 -0.25)
+			(stroke
+				(width 0)
+				(type solid)
+			)
+			(fill solid)
+			(layer "B.SilkS")
+		)
+		(fp_rect
+			(start -2.495672 2.56)
+			(end -1.853977 -0.22)
+			(stroke
+				(width 0)
+				(type solid)
+			)
+			(fill solid)
+			(layer "B.SilkS")
+		)
+		(fp_rect
+			(start -2.495672 0.421695)
+			(end 1.445672 -0.25)
+			(stroke
+				(width 0)
+				(type solid)
+			)
+			(fill solid)
+			(layer "B.SilkS")
+		)
+		(fp_rect
+			(start -5.79 2.57)
+			(end -5.15 -0.24)
+			(stroke
+				(width 0)
+				(type solid)
+			)
+			(fill solid)
+			(layer "B.SilkS")
+		)
+		(fp_rect
+			(start -5.791695 0.421695)
+			(end -2.83 -0.24)
+			(stroke
+				(width 0)
+				(type solid)
+			)
+			(fill solid)
+			(layer "B.SilkS")
+		)
+		(fp_rect
+			(start -9.901695 2.561344)
+			(end -9.26 -0.19)
+			(stroke
+				(width 0)
+				(type solid)
+			)
+			(fill solid)
+			(layer "B.SilkS")
+		)
+		(fp_rect
+			(start -9.902452 2.562703)
+			(end -6.481108 1.921008)
+			(stroke
+				(width 0)
+				(type solid)
+			)
+			(fill solid)
+			(layer "B.SilkS")
+		)
+		(fp_rect
+			(start -9.902452 1.495476)
+			(end -6.481108 0.853781)
+			(stroke
+				(width 0)
+				(type solid)
+			)
+			(fill solid)
+			(layer "B.SilkS")
+		)
+		(fp_rect
+			(start -11.414237 -2.130672)
+			(end 11.414238 -2.77479)
+			(stroke
+				(width 0)
+				(type solid)
+			)
+			(fill solid)
+			(layer "B.SilkS")
+		)
+		(fp_rect
+			(start -11.414237 -3.411344)
+			(end 11.414238 -4.055462)
+			(stroke
+				(width 0)
+				(type solid)
+			)
+			(fill solid)
+			(layer "B.SilkS")
+		)
+		(fp_poly
+			(pts
+				(xy 11.408475 1.173949) (xy 11.408475 -1.494118) (xy 0 -1.494118) (xy -11.408474 -1.494118) (xy -11.408474 1.173949)
+				(xy -10.762712 1.173949) (xy -10.762712 -0.853782) (xy 0 -0.853782) (xy 10.762712 -0.853782) (xy 10.762712 1.173949)
+				(xy 10.762712 3.20168) (xy 0 3.20168) (xy -10.762712 3.20168) (xy -10.762712 1.173949) (xy -11.408474 1.173949)
+				(xy -11.408474 3.842016) (xy 0 3.842016) (xy 11.408475 3.842016)
+			)
+			(stroke
+				(width 0)
+				(type solid)
+			)
+			(fill solid)
+			(layer "B.SilkS")
+		)
+		(fp_poly
+			(pts
+				(xy 2.78 2.09) (xy 2.85 1.99) (xy 2.88 1.53) (xy 3.79 2.1) (xy 4.419371 2.5) (xy 4.58 2.6) (xy 5.124592 2.6)
+				(xy 5.39 2.6) (xy 5.39 2.43) (xy 5.15 2.25) (xy 4.658413 1.92) (xy 3.612589 1.251045) (xy 4.758781 0.5188)
+				(xy 5.356583 0.125377) (xy 5.61 -0.02) (xy 5.61 -0.21) (xy 5.34 -0.21) (xy 4.73 -0.21) (xy 4.099731 0.151404)
+				(xy 3.982203 0.213445) (xy 3.479113 0.481116) (xy 3.156253 0.629659) (xy 2.914639 0.760336) (xy 2.832382 0.580789)
+				(xy 2.78 0.2) (xy 2.77 -0.01) (xy 2.61 -0.04) (xy 2.49 -0.03) (xy 2.46 0.12) (xy 2.45 0.66) (xy 2.43 1.13)
+				(xy 2.37 1.86) (xy 2.37 2.02) (xy 2.47 2.09) (xy 2.59 2.1)
+			)
+			(stroke
+				(width 0)
+				(type solid)
+			)
+			(fill solid)
+			(layer "B.SilkS")
+		)
+		(fp_poly
+			(pts
+				(xy 9 2.56) (xy 9.546617 2.56) (xy 9.89 2.56) (xy 9.89 2.24) (xy 9.89 1.88) (xy 9.47452 1.88) (xy 8.820081 1.88)
+				(xy 8.502542 1.88) (xy 7.77 1.88) (xy 7.09 1.88) (xy 7.09 1.72) (xy 7.09 1.53) (xy 7.824763 1.53)
+				(xy 8.51 1.53) (xy 9.29 1.53) (xy 9.72 1.53) (xy 9.9 1.53) (xy 9.901695 1.173949) (xy 9.9 0.83)
+				(xy 9.48 0.83) (xy 8.92 0.83) (xy 8.502542 0.83) (xy 7.78 0.83) (xy 7.1 0.83) (xy 7.1 0.64) (xy 7.1 0.45)
+				(xy 7.824763 0.452433) (xy 8.51 0.45) (xy 9.31 0.45) (xy 9.9 0.45) (xy 9.9 0.27) (xy 9.901695 0.106722)
+				(xy 9.9 -0.21) (xy 9.65 -0.21) (xy 8.97366 -0.21) (xy 8.072034 -0.213446) (xy 6.242373 -0.213446)
+				(xy 6.242373 1.173949) (xy 6.242373 2.561344) (xy 8.07 2.561344)
+			)
+			(stroke
+				(width 0)
+				(type solid)
+			)
+			(fill solid)
+			(layer "B.SilkS")
 		)
-		(fill none)
-		(layer "F.SilkS")
 	)
 	(gr_rect
@@
 		(layer "Edge.Cuts")
 	)
+	(gr_poly
+		(pts
+			(xy 239.117726 151.365) (xy 237.117726 131.365) (xy 187.117726 131.365) (xy 185.117726 151.365)
+		)
+		(stroke
+			(width 0.2)
+			(type dash_dot_dot)
+		)
+		(fill none)
+		(layer "F.Fab")
+	)
+	(gr_text "8060A LED Mod Rev. 1 - Thanks to all at EEVBlog and ModemHead\nInspired by Dmitri and the original LED 8060A Mod\nPCB Made by Parabolic Labs"
+		(at 243.95 130.83 0)
+		(layer "B.SilkS")
+		(effects
+			(font
+				(size 1 1)
+				(thickness 0.25)
+				(bold yes)
+			)
+			(justify left bottom mirror)
+		)
+	)
 	(segment
